File: ebus_adapter.kicad_sch (KiCad schematic)
At the start: 49 parts, among them J1 KF2EDGK, J2 Conn_01x05_Male, J3 USB_C_Receptacle_USB2.0, J4 Conn_02x02_Top_Bottom, Q1 BC817-40, U1 ME3116, U2 LMV358, U3 ESP32-C3-MINI-1*2

Commit message: Daily save
Parts:
- removed J3: USB_C_Receptacle_USB2.0, Connector_USB:USB_C_Receptacle_Palconn_UTC16-G, symbol Connector:USB_C_Receptacle_USB2.0
- removed J4: Conn_02x02_Top_Bottom, Connector_PinHeader_2.00mm:PinHeader_2x02_P2.00mm_Vertical, symbol Connector_Generic:Conn_02x02_Top_Bottom
- added C8: 100nF, Capacitor_SMD:C_0603_1608Metric, symbol Device:C
- added IC1: FT231XS-R, footprints:SOP63P599X175-20N, symbol robomow_usb-eagle-import:FT231XS-R
- added J5: USB4105-GF-A, footprints:GCT_USB4105-GF-A_1, symbol USB4105-GF-A:USB4105-GF-A
- added R23, R24, R25, R26: 0, Resistor_SMD:R_0603_1608Metric, symbol Device:R
- added U4: USBLC6-2SC6, Package_TO_SOT_SMD:SOT-23-6, symbol Power_Protection:USBLC6-2SC6
- J2: value Conn_01x05_Male -> ESP32 ext programmer
- R16, R18, R9: value 2k2 -> 4K7
- renumbered R21 to R14, R14 to R21
Connections:
- net +3V3: now also C8.1, IC1.13 (3V3OUT), IC1.3 (VCCIO)
- net FROM-EBUS: now also U3.30 (GPIO20/U0RXD), IC1.4 (RXD); no longer U3.31 (GPIO21/U0TXD)
- net GND: now also R14.2, R21.1, C8.2, IC1.16 (GND@2), IC1.6 (GND@1), J5.A1_B12 (GND), J5.B1_A12 (GND), J5.S1 (SHELL_GND), J5.S2 (SHELL_GND), J5.S3 (SHELL_GND), J5.S4 (SHELL_GND), U4.2 (GND); no longer R14.1, R21.2
- net TO-EBUS: now also U3.31 (GPIO21/U0TXD), IC1.20 (TXD); no longer U3.30 (GPIO20/U0RXD)
- net USB_DN: now also J5.A7 (DN1), J5.B7 (DN2), U4.4 (I/O2); no longer U3.26 (GPIO18/USB_D-)
- net USB_DP: now also J5.A6 (DP1), J5.B6 (DP2), U4.6 (I/O1); no longer U3.27 (GPIO19/USB_D+)
- net VBUS: now also D9.2 (A), J5.A4_B9 (VBUS), J5.B4_A9 (VBUS), U4.5 (VBUS)
- net VCC: now also IC1.15 (VCC)
- net TO_ESP: no longer names the net of D1.1 (K), R13.1, U2.1
- new net: J5.A5 (CC1), R14.1
- new net: J5.B5 (CC2), R21.2
- new net USB_DN_ESP: R26.1, U3.26 (GPIO18/USB_D-)
- new net USB_DN_FTDI: IC1.12 (USBDM), R24.1
- new net USB_DN_PROT: R24.2, R26.2, U4.3 (I/O2)
- new net USB_DP_ESP: R25.1, U3.27 (GPIO19/USB_D+)
- new net USB_DP_FTDI: IC1.11 (USBDP), R23.1
- new net USB_DP_PROT: R23.2, R25.2, U4.1 (I/O1)
- no-connect marks 0 -> 19
Other:
- note removed: "ToDO:"
- moved on the sheet: C1, C2, C3, C4, C6, C7, D6, D8, L1, R12, R13, R14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
